File: shema/sh.brd (EAGLE design)
At the start: 37.8 x 71.1 mm, 16 parts, among them X1 X1, X2 X2, X3 X3, X4 X4, X5 x5, X6 x6, Y1 Y1, Y2 Y2, Y3 Y3

Commit message: ~
Parts:
- moved OUT+ 35.6 mm to (24.1, 63.5)
- moved OUT- 29.9 mm to (24.1, 57.1)
- moved IN+ 26.2 mm to (24.1, 44.5)
- moved IN- 16.3 mm to (24.1, 38.1)
- moved Y1 5.68 mm to (33.0, 43.2)
- moved Y2 4.58 mm to (33.0, 53.3)
- moved Y3 3.59 mm to (33.0, 63.5)
- moved C2 2.84 mm to (15.2, 72.4)
- moved C1 2.84 mm to (26.7, 72.4)
- moved IN 2.54 mm to (5.08, 72.4)
Routing:
- net GND: track 239.8 -> 186.8 mm
- net N$3: track 76.2 -> 57.3 mm
- net VCC: track 98.8 -> 94.2 mm
Other:
- board size 37.8 x 71.1 mm -> 46.7 x 47.5 mm
